Commit message: add ros2 control to wrs_env test and controllers

File: src/wrs_cell_description/urdf/wrs_env.urdf.xacro (robot description, xacro)
@@ -113,3 +113,138 @@
         <mu2>0.9</mu2>
     </gazebo>
+    <ros2_control name="RobotSystem" type="system">
+        <hardware>
+            <plugin>gazebo_ros2_control/GazeboSystem</plugin>
+        </hardware>
+        <!-- Joints for packing_arm_ -->
+        <joint name="packing_arm_shoulder_pan_joint">
+            <command_interface name="position">
+                <param name="min">-6.28318530718</param>
+                <param name="max">6.28318530718</param>
+            </command_interface>
+            <state_interface name="position"/>
+            <state_interface name="velocity"/>
+            <state_interface name="effort"/>
+        </joint>
+        <joint name="packing_arm_shoulder_lift_joint">
+            <command_interface name="position">
+                <param name="min">-6.28318530718</param>
+                <param name="max">6.28318530718</param>
+            </command_interface>
+            <state_interface name="position"/>
+            <state_interface name="velocity"/>
+            <state_interface name="effort"/>
+        </joint>
+        <joint name="packing_arm_elbow_joint">
+            <command_interface name="position">
+                <param name="min">-3.14159265359</param>
+                <param name="max">3.14159265359</param>
+            </command_interface>
+            <state_interface name="position"/>
+            <state_interface name="velocity"/>
+            <state_interface name="effort"/>
+        </joint>
+        <joint name="packing_arm_wrist_1_joint">
+            <command_interface name="position">
+                <param name="min">-6.28318530718</param>
+                <param name="max">6.28318530718</param>
+            </command_interface>
+            <state_interface name="position"/>
+            <state_interface name="velocity"/>
+            <state_interface name="effort"/>
+        </joint>
+        <joint name="packing_arm_wrist_2_joint">
+            <command_interface name="position">
+                <param name="min">-6.28318530718</param>
+                <param name="max">6.28318530718</param>
+            </command_interface>
+            <state_interface name="position"/>
+            <state_interface name="velocity"/>
+            <state_interface name="effort"/>
+        </joint>
+        <joint name="packing_arm_wrist_3_joint">
+            <command_interface name="position">
+                <param name="min">-6.28318530718</param>
+                <param name="max">6.28318530718</param>
+            </command_interface>
+            <state_interface name="position"/>
+            <state_interface name="velocity"/>
+            <state_interface name="effort"/>
+        </joint>
+        <!-- Robotiq Gripper Joint for packing_arm_ -->
+        <joint name="packing_arm_robotiq_85_left_knuckle_joint">
+            <command_interface name="position">
+                <param name="min">0.0</param>
+                <param name="max">0.80285</param>
+            </command_interface>
+            <state_interface name="position"/>
+            <state_interface name="velocity"/>
+            <state_interface name="effort"/>
+        </joint>
+        <!-- Joints for cb_ (Cardboard Arm) -->
+        <joint name="cb_shoulder_pan_joint">
+            <command_interface name="position">
+                <param name="min">-6.28318530718</param>
+                <param name="max">6.28318530718</param>
+            </command_interface>
+            <state_interface name="position"/>
+            <state_interface name="velocity"/>
+            <state_interface name="effort"/>
+        </joint>
+        <joint name="cb_shoulder_lift_joint">
+            <command_interface name="position">
+                <param name="min">-6.28318530718</param>
+                <param name="max">6.28318530718</param>
+            </command_interface>
+            <state_interface name="position"/>
+            <state_interface name="velocity"/>
+            <state_interface name="effort"/>
+        </joint>
+        <joint name="cb_elbow_joint">
+            <command_interface name="position">
+                <param name="min">-3.14159265359</param>
+                <param name="max">3.14159265359</param>
+            </command_interface>
+            <state_interface name="position"/>
+            <state_interface name="velocity"/>
+            <state_interface name="effort"/>
+        </joint>
+        <joint name="cb_wrist_1_joint">
+            <command_interface name="position">
+                <param name="min">-6.28318530718</param>
+                <param name="max">6.28318530718</param>
+            </command_interface>
+            <state_interface name="position"/>
+            <state_interface name="velocity"/>
+            <state_interface name="effort"/>
+        </joint>
+        <joint name="cb_wrist_2_joint">
+            <command_interface name="position">
+                <param name="min">-6.28318530718</param>
+                <param name="max">6.28318530718</param>
+            </command_interface>
+            <state_interface name="position"/>
+            <state_interface name="velocity"/>
+            <state_interface name="effort"/>
+        </joint>
+        <joint name="cb_wrist_3_joint">
+            <command_interface name="position">
+                <param name="min">-6.28318530718</param>
+                <param name="max">6.28318530718</param>
+            </command_interface>
+            <state_interface name="position"/>
+            <state_interface name="velocity"/>
+            <state_interface name="effort"/>
+        </joint>
+        <!-- Cardboard Gripper Joint for cb_ -->
+        <joint name="cb_gripper_base_to_finger">
+            <command_interface name="position">
+                <param name="min">0.0</param>
+                <param name="max">1.5708</param>
+            </command_interface>
+            <state_interface name="position"/>
+            <state_interface name="velocity"/>
+            <state_interface name="effort"/>
+        </joint>
+    </ros2_control>
 </robot>

Commit message: more updates

File: src/wrs_cell_description/urdf/wrs_env.urdf.xacro (robot description, xacro)
@@ -7,4 +7,10 @@
     <!-- ur5 -->
     <xacro:include filename="$(find robot_description)/urdf/ur5.urdf.xacro" />
+    <!-- gripper -->
+    <xacro:include filename="$(find robot_description)/urdf/robotiq/robotiq_85_gripper.urdf.xacro" />
+    <!-- cardboard gripper -->
+    <xacro:include filename="$(find cardboard_gripper_description)/gripper/gripper.urdf.xacro" />
+    <!-- World link -->
+    <link name="world" />
     <link name="arm_mount_link" >
         <visual>
@@ -26,16 +32,11 @@
     <!-- arm 1 -->
     <xacro:ur5_robot prefix="${arm_1_prefix}" joint_limited="false"/>
-    <link name="world" />
     <joint name="world_${arm_1_prefix}joint" type="fixed">
         <parent link="world" />
         <child link = "${arm_1_prefix}base_link" />
-        <!-- <origin xyz="0.0 0.23134 0.65866" rpy="${-3*pi/4} 0.0 0.0" /> -->
-        <origin xyz="0.0 0.3 0.65866" rpy="${-3*pi} 0.0 0.0" />
-    </joint>
-    <xacro:include filename="$(find robot_description)/urdf/robotiq/robotiq_85_gripper.urdf.xacro" />
+        <origin xyz="0.0 0.3 0.65866" rpy="${pi} 0.0 0.0" />
+    </joint>
     <!-- Robotiq Coupler -->
-    <!--  + Height added by the coupler: 8mm -->
-    <!--  + Reference frame: at the middle (4mm) -->
-    <link name="robotiq_coupler">
+    <link name="${arm_1_prefix}robotiq_coupler">
     <visual>
         <geometry>
@@ -58,13 +59,13 @@
         <origin xyz="0 0 0.0" rpy="0 0 ${-pi/2.0}" />
         <parent link="${arm_1_prefix}tool0"/>
-        <child link="robotiq_coupler"/>
-    </joint>
-    <gazebo reference="robotiq_coupler">
+        <child link="${arm_1_prefix}robotiq_coupler"/>
+    </joint>
+    <gazebo reference="${arm_1_prefix}robotiq_coupler">
     <mu1>0.9</mu1>
     <mu2>0.9</mu2>
     </gazebo>
     <!-- Attach the robotiq 85 gripper -->
-    <xacro:robotiq_85_gripper prefix="" parent="robotiq_coupler" >
-    <origin xyz="0 0 0.005" rpy="0 ${-pi/2} ${pi/2}"/>
+    <xacro:robotiq_85_gripper prefix="${arm_1_prefix}" parent="${arm_1_prefix}robotiq_coupler" >
+        <origin xyz="0 0 0.005" rpy="0 ${-pi/2} ${pi/2}"/>
     </xacro:robotiq_85_gripper>
     <!-- CardBoard Packing Arm -->
@@ -72,14 +73,11 @@
     <xacro:ur5_robot prefix="${arm_2_prefix}" joint_limited="false"/>
     <!-- Add the gripper -->
-    <xacro:include filename="$(find cardboard_gripper_description)/gripper/gripper.urdf.xacro" />
     <xacro:cardboard_gripper parent="${arm_2_prefix}ee_link" />
     <joint name="world_${arm_2_prefix}joint" type="fixed">
         <parent link="world" />
         <child link = "${arm_2_prefix}base_link" />
-        <!--origin xyz="0.0 -0.23134 0.65866" rpy="${3*pi/4} 0.0 0.0" /--> <!-- for the 45-degree config -->
         <origin xyz="0.0 -0.3 0.65866" rpy="${pi} 0.0 ${pi}" />
     </joint>
     <!-- Add a table as a ground -->
-    <!-- Table -->
     <link name="table">
         <visual>

Commit message: remove controllers

File: src/wrs_cell_description/urdf/wrs_env.urdf.xacro (robot description, xacro)
@@ -111,138 +111,3 @@
         <mu2>0.9</mu2>
     </gazebo>
-    <ros2_control name="RobotSystem" type="system">
-        <hardware>
-            <plugin>gazebo_ros2_control/GazeboSystem</plugin>
-        </hardware>
-        <!-- Joints for packing_arm_ -->
-        <joint name="packing_arm_shoulder_pan_joint">
-            <command_interface name="position">
-                <param name="min">-6.28318530718</param>
-                <param name="max">6.28318530718</param>
-            </command_interface>
-            <state_interface name="position"/>
-            <state_interface name="velocity"/>
-            <state_interface name="effort"/>
-        </joint>
-        <joint name="packing_arm_shoulder_lift_joint">
-            <command_interface name="position">
-                <param name="min">-6.28318530718</param>
-                <param name="max">6.28318530718</param>
-            </command_interface>
-            <state_interface name="position"/>
-            <state_interface name="velocity"/>
-            <state_interface name="effort"/>
-        </joint>
-        <joint name="packing_arm_elbow_joint">
-            <command_interface name="position">
-                <param name="min">-3.14159265359</param>
-                <param name="max">3.14159265359</param>
-            </command_interface>
-            <state_interface name="position"/>
-            <state_interface name="velocity"/>
-            <state_interface name="effort"/>
-        </joint>
-        <joint name="packing_arm_wrist_1_joint">
-            <command_interface name="position">
-                <param name="min">-6.28318530718</param>
-                <param name="max">6.28318530718</param>
-            </command_interface>
-            <state_interface name="position"/>
-            <state_interface name="velocity"/>
-            <state_interface name="effort"/>
-        </joint>
-        <joint name="packing_arm_wrist_2_joint">
-            <command_interface name="position">
-                <param name="min">-6.28318530718</param>
-                <param name="max">6.28318530718</param>
-            </command_interface>
-            <state_interface name="position"/>
-            <state_interface name="velocity"/>
-            <state_interface name="effort"/>
-        </joint>
-        <joint name="packing_arm_wrist_3_joint">
-            <command_interface name="position">
-                <param name="min">-6.28318530718</param>
-                <param name="max">6.28318530718</param>
-            </command_interface>
-            <state_interface name="position"/>
-            <state_interface name="velocity"/>
-            <state_interface name="effort"/>
-        </joint>
-        <!-- Robotiq Gripper Joint for packing_arm_ -->
-        <joint name="packing_arm_robotiq_85_left_knuckle_joint">
-            <command_interface name="position">
-                <param name="min">0.0</param>
-                <param name="max">0.80285</param>
-            </command_interface>
-            <state_interface name="position"/>
-            <state_interface name="velocity"/>
-            <state_interface name="effort"/>
-        </joint>
-        <!-- Joints for cb_ (Cardboard Arm) -->
-        <joint name="cb_shoulder_pan_joint">
-            <command_interface name="position">
-                <param name="min">-6.28318530718</param>
-                <param name="max">6.28318530718</param>
-            </command_interface>
-            <state_interface name="position"/>
-            <state_interface name="velocity"/>
-            <state_interface name="effort"/>
-        </joint>
-        <joint name="cb_shoulder_lift_joint">
-            <command_interface name="position">
-                <param name="min">-6.28318530718</param>
-                <param name="max">6.28318530718</param>
-            </command_interface>
-            <state_interface name="position"/>
-            <state_interface name="velocity"/>
-            <state_interface name="effort"/>
-        </joint>
-        <joint name="cb_elbow_joint">
-            <command_interface name="position">
-                <param name="min">-3.14159265359</param>
-                <param name="max">3.14159265359</param>
-            </command_interface>
-            <state_interface name="position"/>
-            <state_interface name="velocity"/>
-            <state_interface name="effort"/>
-        </joint>
-        <joint name="cb_wrist_1_joint">
-            <command_interface name="position">
-                <param name="min">-6.28318530718</param>
-                <param name="max">6.28318530718</param>
-            </command_interface>
-            <state_interface name="position"/>
-            <state_interface name="velocity"/>
-            <state_interface name="effort"/>
-        </joint>
-        <joint name="cb_wrist_2_joint">
-            <command_interface name="position">
-                <param name="min">-6.28318530718</param>
-                <param name="max">6.28318530718</param>
-            </command_interface>
-            <state_interface name="position"/>
-            <state_interface name="velocity"/>
-            <state_interface name="effort"/>
-        </joint>
-        <joint name="cb_wrist_3_joint">
-            <command_interface name="position">
-                <param name="min">-6.28318530718</param>
-                <param name="max">6.28318530718</param>
-            </command_interface>
-            <state_interface name="position"/>
-            <state_interface name="velocity"/>
-            <state_interface name="effort"/>
-        </joint>
-        <!-- Cardboard Gripper Joint for cb_ -->
-        <joint name="cb_gripper_base_to_finger">
-            <command_interface name="position">
-                <param name="min">0.0</param>
-                <param name="max">1.5708</param>
-            </command_interface>
-            <state_interface name="position"/>
-            <state_interface name="velocity"/>
-            <state_interface name="effort"/>
-        </joint>
-    </ros2_control>
 </robot>
