Commit message: fix ur5 position

File: src/wrs_cell_description/urdf/wrs_env_V2.urdf.xacro (robot description, xacro)
@@ -40,5 +40,5 @@
         <parent link="robot_base"/>
         <child link="${arm_prefix}base_link"/>
-        <origin xyz="0 0.25 0.2" rpy="0 0 ${pi}"/>
+        <origin xyz="0 0.25 0.31" rpy="0 0 ${pi/2}"/>
     </joint>
     <!-- Robotiq Coupler -->

Commit message: - Replaced the robot table with the  Cobot Station

File: src/wrs_cell_description/urdf/wrs_env_V2.urdf.xacro (robot description, xacro)
@@ -14,17 +14,14 @@
         <visual>
             <geometry>
-                <box size="1.0 0.8 0.4"/>
+                <mesh filename="package://robot_description/meshes/cobot_station/visual/BancaleUR.dae" />
             </geometry>
-            <material name="grey">
-                <color rgba="0.5 0.5 0.5 1.0"/>
-            </material>
         </visual>
         <collision>
             <geometry>
-                <box size="0.8 0.8 0.4"/>
+                <mesh filename="package://robot_description/meshes/cobot_station/collision/BancaleUR_collision.stl" />
             </geometry>
         </collision>
         <inertial>
-            <mass value="50"/>
+            <mass value="275.0"/>
             <origin xyz="0 0 0" rpy="0 0 0"/>
             <inertia ixx="1.0" ixy="0.0" ixz="0.0" iyy="1.0" iyz="0.0" izz="1.0"/>
@@ -34,5 +31,5 @@
         <parent link="world"/>
         <child link="robot_base"/>
-        <origin xyz="0 0 0.2" rpy="0 0 0"/>
+        <origin xyz="0 0 0.0" rpy="0 0 0"/>
     </joint>
     <!-- Attach UR5 to the base -->

Commit message: - Updated URDF configuration to instantiate the UR5e arm using the official macro. - Added fake hardware and sensor commands xacro:args.

File: src/wrs_cell_description/urdf/wrs_env_V2.urdf.xacro (robot description, xacro)
@@ -3,9 +3,25 @@
     <xacro:property name="arm_prefix" value="ur5_"/>
     <!-- ur5 -->
+    <xacro:arg name="use_fake_hardware" default="true"/>
+    <xacro:arg name="fake_sensor_commands" default="true"/>
+    <!-- Include official UR5e description from ur_description package -->
+    <xacro:include filename="$(find ur_description)/urdf/ur_macro.xacro"/>
     <xacro:include filename="$(find robot_description)/urdf/ur5.urdf.xacro" />
     <!-- gripper -->
     <xacro:include filename="$(find robot_description)/urdf/robotiq/robotiq_85_gripper.urdf.xacro" />
     <!-- arm -->
-    <xacro:ur5_robot prefix="${arm_prefix}" joint_limited="false"/>
+    <!-- Instantiate UR5e arm with official macro -->
+    <xacro:ur_robot
+        name="ur5e"
+        tf_prefix="${arm_prefix}"
+        parent="robot_base"
+        use_fake_hardware="$(arg use_fake_hardware)"
+        fake_sensor_commands="$(arg fake_sensor_commands)"
+        joint_limits_parameters_file="$(find ur_description)/config/ur5e/joint_limits.yaml"
+        kinematics_parameters_file="$(find ur_description)/config/ur5e/default_kinematics.yaml"
+        physical_parameters_file="$(find ur_description)/config/ur5e/physical_parameters.yaml"
+        visual_parameters_file="$(find ur_description)/config/ur5e/visual_parameters.yaml">
+        <origin xyz="-0.1 -0.1 0" rpy="0 0 0"/>
+    </xacro:ur_robot>
     <!-- World link -->
     <link name="world" />

Commit message: - Adapted  the dimensions, mass, and pose of conveyor belt in the urdf file.

File: src/wrs_cell_description/urdf/wrs_env_V2.urdf.xacro (robot description, xacro)
@@ -84,8 +84,11 @@
     </xacro:robotiq_85_gripper>
     <!-- Rail -->
+    <xacro:property name="rail_length" value="2.0"/>
+    <xacro:property name="rail_width" value="0.8"/>
+    <xacro:property name="rail_height" value="0.8"/>
     <link name="rail_link">
         <visual>
             <geometry>
-                <box size="2.0 0.8 0.4"/>
+                <box size="${rail_length} ${rail_width} ${rail_height}"/>
             </geometry>
             <material name="dark_grey">
@@ -95,9 +98,9 @@
         <collision>
             <geometry>
-                <box size="2.0 0.8 0.4"/>
+                <box size="${rail_length} ${rail_width} ${rail_height}"/>
             </geometry>
         </collision>
         <inertial>
-            <mass value="10"/>
+            <mass value="100"/>
             <origin xyz="0 0 0" rpy="0 0 0"/>
             <inertia ixx="1.0" ixy="0.0" ixz="0.0" iyy="1.0" iyz="0.0" izz="1.0"/>
@@ -107,5 +110,5 @@
         <parent link="world"/>
         <child link="rail_link"/>
-        <origin xyz="0.4 0.83 0.2" rpy="0 0 0"/>
+        <origin xyz="${rail_width/2 + 0.1} ${0/2} ${-rail_height/2 - 0.1}" rpy="0 0 ${pi/2}"/>
     </joint>
 </robot>

Commit message: - Resolved the problem with URDF file to avoid redundant joint - Add initial positions configuration for wrs_cell_v2 - Modifiled initial position file

File: src/wrs_cell_description/urdf/wrs_env_V2.urdf.xacro (robot description, xacro)
@@ -7,9 +7,10 @@
     <!-- Include official UR5e description from ur_description package -->
     <xacro:include filename="$(find ur_description)/urdf/ur_macro.xacro"/>
-    <xacro:include filename="$(find robot_description)/urdf/ur5.urdf.xacro" />
     <!-- gripper -->
     <xacro:include filename="$(find robot_description)/urdf/robotiq/robotiq_85_gripper.urdf.xacro" />
     <!-- arm -->
     <!-- Instantiate UR5e arm with official macro -->
+    <xacro:arg name="initial_positions_file" default="$(find wrs_env_v2_moveit_config)/config/initial_positions.yaml" />
+    <xacro:property name="initial_positions" value="${xacro.load_yaml('$(arg initial_positions_file)')['initial_positions']}"/>
     <xacro:ur_robot
         name="ur5e"
@@ -21,5 +22,6 @@
         kinematics_parameters_file="$(find ur_description)/config/ur5e/default_kinematics.yaml"
         physical_parameters_file="$(find ur_description)/config/ur5e/physical_parameters.yaml"
-        visual_parameters_file="$(find ur_description)/config/ur5e/visual_parameters.yaml">
+        visual_parameters_file="$(find ur_description)/config/ur5e/visual_parameters.yaml"
+        initial_positions="${initial_positions}">
         <origin xyz="-0.1 -0.1 0" rpy="0 0 0"/>
     </xacro:ur_robot>
@@ -48,10 +50,4 @@
         <child link="robot_base"/>
         <origin xyz="0 0 0.0" rpy="0 0 0"/>
-    </joint>
-    <!-- Attach UR5 to the base -->
-    <joint name="base_to_ur5_joint" type="fixed">
-        <parent link="robot_base"/>
-        <child link="${arm_prefix}base_link"/>
-        <origin xyz="0 0.25 0.31" rpy="0 0 ${pi/2}"/>
     </joint>
     <!-- Robotiq Coupler -->

File: src/wrs_env_v2_moveit_config/config/wrs_cell_v2.urdf.xacro (robot description, xacro)
@@ -1,5 +1,5 @@
 <?xml version="1.0"?>
 <robot xmlns:xacro="http://www.ros.org/wiki/xacro" name="wrs_cell_v2">
-    <xacro:arg name="initial_positions_file" default="initial_positions.yaml" />
+    <xacro:arg name="initial_positions_file" default="$(find wrs_env_v2_moveit_config)/config/initial_positions.yaml" />
     <!-- Import wrs_cell_v2 urdf file -->
     <xacro:include filename="$(find wrs_cell_description)/urdf/wrs_env_V2.urdf.xacro" />

Commit message: add initial adapter

File: src/wrs_cell_description/urdf/wrs_env_V2.urdf.xacro (robot description, xacro)
@@ -51,4 +51,29 @@
         <child link="robot_base"/>
         <origin xyz="0 0 0.0" rpy="0 0 0"/>
+    </joint>
+    <!-- Gripper adapter -->
+    <link name="${arm_prefix}gripper_adapter">
+      <visual>
+        <geometry>
+          <mesh filename="package://robot_description/meshes/gripper_adapter.stl" />
+        </geometry>
+      </visual>
+      <collision>
+        <geometry>
+          <mesh filename="package://robot_description/meshes/gripper_adapter.stl" />
+        </geometry>
+      </collision>
+      <!-- TODO: check inertia -->
+      <inertial>
+        <origin xyz="2.073e-05   1.45286e-03  -1.1049e-03" rpy="0 0 0" />
+        <mass value="0.168" />
+        <inertia ixx="6.69695624e-05" ixy="5.21511788e-09" ixz="-2.74383009e-08"
+                 iyy="7.85088161e-05" iyz="5.41105193e-07" izz="1.41819717e-04"/>
+      </inertial>
+    </link>
+    <joint name="${arm_prefix}gripper_adapter_joint" type="fixed">
+        <origin xyz="0 0 -0.003" rpy="0 0 ${-pi/2.0}" /> <!-- TODO: adapt origin -->
+        <parent link="${arm_prefix}roboti_coupler"/> <!-- ask if it will replace it -->
+      <child link="${arm_prefix}gripper_adapter"/>
     </joint>
     <!-- Robotiq Coupler -->

Commit message: add gripper adapter

File: src/wrs_cell_description/urdf/wrs_env_V2.urdf.xacro (robot description, xacro)
@@ -56,10 +56,10 @@
       <visual>
         <geometry>
-          <mesh filename="package://robot_description/meshes/gripper_adapter.stl" />
+          <mesh filename="package://robot_description/meshes/gripper_adapter.stl" scale="0.001 0.001 0.001"/>
         </geometry>
       </visual>
       <collision>
         <geometry>
-          <mesh filename="package://robot_description/meshes/gripper_adapter.stl" />
+          <mesh filename="package://robot_description/meshes/gripper_adapter.stl" scale="0.001 0.001 0.001"/>
         </geometry>
       </collision>
@@ -73,35 +73,11 @@
     </link>
     <joint name="${arm_prefix}gripper_adapter_joint" type="fixed">
-        <origin xyz="0 0 -0.003" rpy="0 0 ${-pi/2.0}" /> <!-- TODO: adapt origin -->
-        <parent link="${arm_prefix}roboti_coupler"/> <!-- ask if it will replace it -->
+      <origin xyz="0 0 -0.003" rpy="0 0 ${-pi/2.0}" />
+      <parent link="${arm_prefix}tool0"/>
       <child link="${arm_prefix}gripper_adapter"/>
     </joint>
-    <!-- Robotiq Coupler -->
-    <link name="${arm_prefix}robotiq_coupler">
-      <visual>
-        <geometry>
-          <mesh filename="package://robot_description/meshes/suction_base.stl" />
-        </geometry>
-      </visual>
-      <collision>
-        <geometry>
-          <mesh filename="package://robot_description/meshes/suction_base.stl" />
-        </geometry>
-      </collision>
-      <inertial>
-        <origin xyz="2.073e-05   1.45286e-03  -1.1049e-03" rpy="0 0 0" />
-        <mass value="0.168" />
-        <inertia ixx="6.69695624e-05" ixy="5.21511788e-09" ixz="-2.74383009e-08"
-                 iyy="7.85088161e-05" iyz="5.41105193e-07" izz="1.41819717e-04"/>
-      </inertial>
-    </link>
-    <joint name="${arm_prefix}robotiq_coupler_joint" type="fixed">
-      <origin xyz="0 0 -0.003" rpy="0 0 ${-pi/2.0}" />
-      <parent link="${arm_prefix}tool0"/>
-      <child link="${arm_prefix}robotiq_coupler"/>
-    </joint>
     <!-- Attach the robotiq 85 gripper -->
-    <xacro:robotiq_85_gripper prefix="${arm_prefix}" parent="${arm_prefix}robotiq_coupler" >
-      <origin xyz="0 0 0.08" rpy="0 ${-pi/2} ${pi/2}"/>
+    <xacro:robotiq_85_gripper prefix="${arm_prefix}" parent="${arm_prefix}gripper_adapter" >
+        <origin xyz="-0.035 0.0 0.075" rpy="${pi/2} ${-5*pi/6} 0"/>
     </xacro:robotiq_85_gripper>
     <!-- Rail -->

Commit message: - Update gripper adapter with the new stl file - Added Robotiq and suction cup tcp definitions in the urdf file

File: src/wrs_cell_description/urdf/wrs_env_V2.urdf.xacro (robot description, xacro)
@@ -6,8 +6,12 @@
     <xacro:arg name="fake_sensor_commands" default="false"/>
     <xacro:arg name="robot_ip" default="192.168.1.102"/>
+    <!-- gripper tcp offset - from base of the robotiq to tip of the fingers in closed position -->
+    <!-- reference: https://assets.robotiq.com/website-assets/support_documents/document/online/2F-85_2F-140_TM_InstructionManual_HTML5_20190503.zip/2F-85_2F-140_TM_InstructionManual_HTML5/Content/6.%20Specifications.htm -->
+    <xacro:property name="gripper_tcp_offset" value="0.1628" /> <!--might add 14mm if added the coulping piece -->
     <!-- Include official UR5e description from ur_description package -->
     <xacro:include filename="$(find ur_description)/urdf/ur_macro.xacro"/>
     <!-- gripper -->
-    <xacro:include filename="$(find robot_description)/urdf/robotiq/robotiq_85_gripper.urdf.xacro" />
+    <xacro:arg name="com_port" default="/dev/ttyUSB0" />
+    <xacro:include filename="$(find robotiq_description)/urdf/robotiq_2f_85_macro.urdf.xacro" />
     <!-- arm -->
     <!-- Instantiate UR5e arm with official macro -->
@@ -73,12 +77,28 @@
     </link>
     <joint name="${arm_prefix}gripper_adapter_joint" type="fixed">
-      <origin xyz="0 0 -0.003" rpy="0 0 ${-pi/2.0}" />
-      <parent link="${arm_prefix}tool0"/>
+      <origin xyz="-0.006 0 0" rpy="0 ${pi/2.0} 0" />
+      <parent link="${arm_prefix}flange"/>
       <child link="${arm_prefix}gripper_adapter"/>
     </joint>
     <!-- Attach the robotiq 85 gripper -->
-    <xacro:robotiq_85_gripper prefix="${arm_prefix}" parent="${arm_prefix}gripper_adapter" >
-        <origin xyz="-0.035 0.0 0.075" rpy="${pi/2} ${-5*pi/6} 0"/>
-    </xacro:robotiq_85_gripper>
+    <xacro:robotiq_gripper name="RobotiqGripperHardwareInterface" prefix="${arm_prefix}" parent="${arm_prefix}gripper_adapter" use_fake_hardware="$(arg use_fake_hardware)" com_port="$(arg com_port)">
+        <origin xyz="-0.03299 0.0 0.07114" rpy="${0} ${pi/2-5*pi/6} 0"/>
+    </xacro:robotiq_gripper>
+    <!-- Robotiq Gripper Tool Center Point (TCP) - Frame between gripper fingers -->
+    <link name="${arm_prefix}gripper_tcp" />
+    <joint name="${arm_prefix}gripper_tcp_joint" type="fixed">
+        <parent link="${arm_prefix}robotiq_85_base_link"/>
+        <child link="${arm_prefix}gripper_tcp"/>
+        <!-- Position at the center between the gripper fingers -->
+        <origin xyz="0.0 0.0 ${gripper_tcp_offset}" rpy="0 0 0"/>
+    </joint>
+    <!-- Suction Cup Tool Center Point (TCP) - Frame between suction cup -->
+    <link name="${arm_prefix}suction_tcp" />
+    <joint name="${arm_prefix}suction_tcp_joint" type="fixed">
+        <parent link="${arm_prefix}gripper_adapter"/>
+        <child link="${arm_prefix}suction_tcp"/>
+        <!-- Position at the center between the gripper fingers -->
+        <origin xyz="0.03299 0.0 0.07114" rpy="0 ${pi/3} 0"/>
+    </joint>
     <!-- Rail -->
     <xacro:property name="rail_length" value="2.0"/>

Commit message: - Modified the origin of the robot in the URDF to use calculated values for better positioning.

File: src/wrs_cell_description/urdf/wrs_env_V2.urdf.xacro (robot description, xacro)
@@ -29,5 +29,5 @@
         visual_parameters_file="$(find ur_description)/config/ur5e/visual_parameters.yaml"
         initial_positions="${initial_positions}">
-        <origin xyz="-0.1 -0.1 0" rpy="0 0 0"/>
+        <origin xyz="${-0.27/2} ${-0.27/2} 0.015" rpy="0 0 0"/>
     </xacro:ur_robot>
     <!-- World link -->
@@ -54,5 +54,5 @@
         <parent link="world"/>
         <child link="robot_base"/>
-        <origin xyz="0 0 0.0" rpy="0 0 0"/>
+        <origin xyz="0 0 0" rpy="0 0 0"/>
     </joint>
     <!-- Gripper adapter -->

Commit message: Update URDF and RViz configuration for camera integration
- Modified the URDF to include a camera pillar and camera link with appropriate joints.
- Adjusted the origin of the flange joint to be consistent with the real hardware installation.
- Updated the RViz configuration to visualize the new camera components and adjusted various display settings for better usability.

File: src/wrs_cell_description/urdf/wrs_env_V2.urdf.xacro (robot description, xacro)
@@ -29,5 +29,5 @@
         visual_parameters_file="$(find ur_description)/config/ur5e/visual_parameters.yaml"
         initial_positions="${initial_positions}">
-        <origin xyz="${-0.27/2} ${-0.27/2} 0.015" rpy="0 0 0"/>
+        <origin xyz="${-0.27/2} ${-0.27/2} 0.015" rpy="0 0 ${pi}"/>
     </xacro:ur_robot>
     <!-- World link -->
@@ -56,4 +56,10 @@
         <origin xyz="0 0 0" rpy="0 0 0"/>
     </joint>
+    <link name="${arm_prefix}flange_rotated_link" />
+    <joint name="${arm_prefix}flange_rotated_joint" type="fixed">
+        <parent link="${arm_prefix}flange"/>
+        <child link="${arm_prefix}flange_rotated_link"/>
+        <origin xyz="0 0 0" rpy="${pi/2.0} 0 0"/>
+    </joint>
     <!-- Gripper adapter -->
     <link name="${arm_prefix}gripper_adapter">
@@ -78,5 +84,5 @@
     <joint name="${arm_prefix}gripper_adapter_joint" type="fixed">
       <origin xyz="-0.006 0 0" rpy="0 ${pi/2.0} 0" />
-      <parent link="${arm_prefix}flange"/>
+      <parent link="${arm_prefix}flange_rotated_link"/>
       <child link="${arm_prefix}gripper_adapter"/>
     </joint>
@@ -100,4 +106,29 @@
         <!-- Position at the center between the gripper fingers -->
         <origin xyz="0.03299 0.0 0.07114" rpy="0 ${pi/3} 0"/>
+    </joint>
+    <!-- add camera pillar -->
+    <link name="camera_pillar_link" >
+        <visual>
+            <geometry>
+                <box size="0.08 0.08 0.997"/>
+            </geometry>
+        </visual>
+        <collision>
+            <geometry>
+                <box size="0.08 0.08 0.997"/>
+            </geometry>
+        </collision>
+    </link>
+    <joint name="camera_pillar_joint" type="fixed">
+        <parent link="world"/>
+        <child link="camera_pillar_link"/>
+        <origin xyz="-0.06 -0.96 0.0" rpy="0 0 0"/>
+    </joint>
+    <!-- define camera link -->
+    <link name="camera_link" />
+    <joint name="camera_to_worldjoint" type="fixed">
+        <parent link="camera_pillar_link"/>
+        <child link="camera_link"/>
+        <origin xyz="-0.06 -0.96 1.0" rpy="0 0 0"/>
     </joint>
     <!-- Rail -->

Commit message: Add suction gripper model to URDF
- Introduced new STL files for the suction gripper's visual and collision representations.
- Updated the URDF to include the suction gripper with its mounting frame and joint configurations.
- Defined properties for the suction cup thickness and adjusted the TCP joint origin accordingly.

File: src/wrs_cell_description/urdf/wrs_env_V2.urdf.xacro (robot description, xacro)
@@ -9,4 +9,6 @@
     <!-- reference: https://assets.robotiq.com/website-assets/support_documents/document/online/2F-85_2F-140_TM_InstructionManual_HTML5_20190503.zip/2F-85_2F-140_TM_InstructionManual_HTML5/Content/6.%20Specifications.htm -->
     <xacro:property name="gripper_tcp_offset" value="0.1628" /> <!--might add 14mm if added the coulping piece -->
+    <!-- suction gripper properties -->
+    <xacro:property name="thickness_of_the_suction_cup" value="0.030" /> <!-- 30mm -->
     <!-- Include official UR5e description from ur_description package -->
     <xacro:include filename="$(find ur_description)/urdf/ur_macro.xacro"/>
@@ -99,11 +101,41 @@
         <origin xyz="0.0 0.0 ${gripper_tcp_offset}" rpy="0 0 0"/>
     </joint>
+    <!-- suction gripper mount frame - represents the position of the center of the branch to which the suction gripper is mounted -->
+    <link name="${arm_prefix}suction_gripper_mount_frame" />
+    <joint name="${arm_prefix}suction_gripper_mount_frame_joint" type="fixed">
+        <parent link="${arm_prefix}flange_rotated_link"/>
+        <child link="${arm_prefix}suction_gripper_mount_frame"/>
+        <origin xyz="0.065141 0.0 -0.03299" rpy="0 ${pi/2 + pi/3} 0"/>
+    </joint>
+    <!-- add suction gripper  -->
+    <link name="${arm_prefix}suction_gripper" >
+        <visual>
+            <geometry>
+                <mesh filename="package://robot_description/meshes/suction_gripper/visual/suction_gripper.stl" />
+            </geometry>
+        </visual>
+        <collision>
+            <geometry>
+                <mesh filename="package://robot_description/meshes/suction_gripper/collision/suction_gripper.stl" />
+            </geometry>
+        </collision>
+        <inertial>
+            <origin xyz="0.0 0.0 0.0" rpy="0 0 0"/>
+            <mass value="0.2" />
+            <inertia ixx="0.00001" ixy="0.000000" ixz="0.000000"
+                     iyy="0.00001" iyz="0.000000" izz="0.00001"/>
+        </inertial>
+    </link>
+    <joint name="${arm_prefix}suction_gripper_joint" type="fixed">
+        <parent link="${arm_prefix}suction_gripper_mount_frame"/>
+        <child link="${arm_prefix}suction_gripper"/>
+        <origin xyz="0.0 0.0 -0.0065" rpy="0 0 0"/>
+    </joint>
     <!-- Suction Cup Tool Center Point (TCP) - Frame between suction cup -->
     <link name="${arm_prefix}suction_tcp" />
     <joint name="${arm_prefix}suction_tcp_joint" type="fixed">
-        <parent link="${arm_prefix}gripper_adapter"/>
+        <parent link="${arm_prefix}suction_gripper"/>
         <child link="${arm_prefix}suction_tcp"/>
-        <!-- Position at the center between the gripper fingers -->
-        <origin xyz="0.03299 0.0 0.07114" rpy="0 ${pi/3} 0"/>
+        <origin xyz="0 0 ${0.144 + thickness_of_the_suction_cup}" rpy="0 0 0"/>
     </joint>
     <!-- add camera pillar -->
