Commit message: adapted the urdf file with 2f180 gripper

File: src/wrs_cell_description/urdf/wrs_env_V2.urdf.xacro (robot description, xacro)
@@ -6,7 +6,4 @@
     <xacro:arg name="fake_sensor_commands" default="false"/>
     <xacro:arg name="robot_ip" default="192.168.1.102"/>
-    <!-- gripper tcp offset - from base of the robotiq to tip of the fingers in closed position -->
-    <!-- reference: https://assets.robotiq.com/website-assets/support_documents/document/online/2F-85_2F-140_TM_InstructionManual_HTML5_20190503.zip/2F-85_2F-140_TM_InstructionManual_HTML5/Content/6.%20Specifications.htm -->
-    <xacro:property name="gripper_tcp_offset" value="0.1628" /> <!--might add 14mm if added the coulping piece -->
     <!-- suction gripper properties -->
     <xacro:property name="thickness_of_the_suction_cup" value="0.030" /> <!-- 30mm -->
@@ -15,5 +12,4 @@
     <!-- gripper -->
     <xacro:arg name="com_port" default="/dev/ttyUSB0" />
-    <xacro:include filename="$(find robotiq_description)/urdf/robotiq_2f_85_macro.urdf.xacro" />
     <!-- arm -->
     <!-- Instantiate UR5e arm with official macro -->
@@ -76,5 +72,4 @@
         </geometry>
       </collision>
-      <!-- TODO: check inertia -->
       <inertial>
         <origin xyz="2.073e-05   1.45286e-03  -1.1049e-03" rpy="0 0 0" />
@@ -89,15 +84,27 @@
       <child link="${arm_prefix}gripper_adapter"/>
     </joint>
-    <!-- Attach the robotiq 85 gripper -->
-    <xacro:robotiq_gripper name="RobotiqGripperHardwareInterface" prefix="${arm_prefix}" parent="${arm_prefix}gripper_adapter" use_fake_hardware="$(arg use_fake_hardware)" com_port="$(arg com_port)">
-        <origin xyz="-0.03299 0.0 0.07114" rpy="${0} ${pi/2-5*pi/6} 0"/>
+    <!-- ======================================== Robotiq gripper ======================================== -->
+    <link name="${arm_prefix}robotiq_attaching_point" />
+    <!-- gripper tcp offset - from base of the robotiq to tip of the fingers in closed position -->
+    <!-- reference: https://assets.robotiq.com/website-assets/support_documents/document/online/2F-85_2F-140_TM_InstructionManual_HTML5_20190503.zip/2F-85_2F-140_TM_InstructionManual_HTML5/Content/6.%20Specifications.htm -->
+    <xacro:property name="gripper_tcp_offset" value="0.2333" /> <!--without coupling thickness -->
+    <xacro:property name="robotiq_coupling_thickness" value="0.0169" />
+    <joint name="${arm_prefix}robotiq_attaching_point_joint" type="fixed">
+        <parent link="${arm_prefix}gripper_adapter"/>
+        <child link="${arm_prefix}robotiq_attaching_point"/>
+        <origin xyz="-0.03299 0.0 0.07114" rpy="0 -${pi/3} 0"/>
+    </joint>
+    <!-- <xacro:include filename="$(find robotiq_description)/urdf/robotiq_2f_85_macro.urdf.xacro" /> -->
+    <xacro:include filename="$(find robotiq_description)/urdf/robotiq_2f_140_macro.urdf.xacro" />
+    <xacro:robotiq_gripper name="RobotiqGripperHardwareInterface" prefix="${arm_prefix}" parent="${arm_prefix}robotiq_attaching_point" use_fake_hardware="$(arg use_fake_hardware)" com_port="$(arg com_port)">
+        <origin xyz="0 0 ${robotiq_coupling_thickness}" rpy="0 0 0"/>
     </xacro:robotiq_gripper>
     <!-- Robotiq Gripper Tool Center Point (TCP) - Frame between gripper fingers -->
     <link name="${arm_prefix}gripper_tcp" />
     <joint name="${arm_prefix}gripper_tcp_joint" type="fixed">
-        <parent link="${arm_prefix}robotiq_85_base_link"/>
+        <parent link="${arm_prefix}robotiq_base_link"/>
         <child link="${arm_prefix}gripper_tcp"/>
         <!-- Position at the center between the gripper fingers -->
-        <origin xyz="0.0 0.0 ${gripper_tcp_offset}" rpy="0 0 0"/>
+        <origin xyz="0.0 0.0 ${gripper_tcp_offset + robotiq_coupling_thickness}" rpy="0 0 0"/>
     </joint>
     <!-- suction gripper mount frame - represents the position of the center of the branch to which the suction gripper is mounted -->

Commit message: replaced the gripper adapter with the 90-deg one; corrected and checked all the link frames in the urdf file

File: src/wrs_cell_description/urdf/wrs_env_V2.urdf.xacro (robot description, xacro)
@@ -12,4 +12,6 @@
     <!-- gripper -->
     <xacro:arg name="com_port" default="/dev/ttyUSB0" />
+    <!-- cobot station height-->
+    <xacro:property name="cobot_station_height" value="0.91"/>
     <!-- arm -->
     <!-- Instantiate UR5e arm with official macro -->
@@ -80,5 +82,5 @@
     </link>
     <joint name="${arm_prefix}gripper_adapter_joint" type="fixed">
-      <origin xyz="-0.006 0 0" rpy="0 ${pi/2.0} 0" />
+      <origin xyz="-0.006 0 0" rpy="0 ${pi/2} 0" />
       <parent link="${arm_prefix}flange_rotated_link"/>
       <child link="${arm_prefix}gripper_adapter"/>
@@ -91,27 +93,29 @@
     <xacro:property name="robotiq_coupling_thickness" value="0.0169" />
     <joint name="${arm_prefix}robotiq_attaching_point_joint" type="fixed">
-        <parent link="${arm_prefix}gripper_adapter"/>
+        <parent link="${arm_prefix}flange_rotated_link"/>
         <child link="${arm_prefix}robotiq_attaching_point"/>
-        <origin xyz="-0.03299 0.0 0.07114" rpy="0 -${pi/3} 0"/>
+        <origin xyz="0.052123 0.0 0.037123" rpy="0 -${pi/4} 0"/>
     </joint>
     <!-- <xacro:include filename="$(find robotiq_description)/urdf/robotiq_2f_85_macro.urdf.xacro" /> -->
     <xacro:include filename="$(find robotiq_description)/urdf/robotiq_2f_140_macro.urdf.xacro" />
-    <xacro:robotiq_gripper name="RobotiqGripperHardwareInterface" prefix="${arm_prefix}" parent="${arm_prefix}robotiq_attaching_point" use_fake_hardware="$(arg use_fake_hardware)" com_port="$(arg com_port)">
-        <origin xyz="0 0 ${robotiq_coupling_thickness}" rpy="0 0 0"/>
+    <xacro:robotiq_gripper name="RobotiqGripperHardwareInterface" prefix="${arm_prefix}"
+        parent="${arm_prefix}robotiq_attaching_point" use_fake_hardware="$(arg use_fake_hardware)" com_port="$(arg com_port)">
+        <origin xyz="0 ${-robotiq_coupling_thickness} 0" rpy="${pi/2} 0 0"/>
     </xacro:robotiq_gripper>
     <!-- Robotiq Gripper Tool Center Point (TCP) - Frame between gripper fingers -->
     <link name="${arm_prefix}gripper_tcp" />
     <joint name="${arm_prefix}gripper_tcp_joint" type="fixed">
-        <parent link="${arm_prefix}robotiq_base_link"/>
+        <parent link="${arm_prefix}robotiq_attaching_point"/>
         <child link="${arm_prefix}gripper_tcp"/>
         <!-- Position at the center between the gripper fingers -->
-        <origin xyz="0.0 0.0 ${gripper_tcp_offset + robotiq_coupling_thickness}" rpy="0 0 0"/>
+        <!--origin xyz="0.0 0.0 0.252" rpy="0 0 0"/> TODO: hardcoded value -->
+        <origin xyz="${gripper_tcp_offset + robotiq_coupling_thickness} 0 0" rpy="0 ${pi/2} 0"/>
     </joint>
     <!-- suction gripper mount frame - represents the position of the center of the branch to which the suction gripper is mounted -->
-    <link name="${arm_prefix}suction_gripper_mount_frame" />
-    <joint name="${arm_prefix}suction_gripper_mount_frame_joint" type="fixed">
+    <link name="${arm_prefix}suction_gripper_attaching_point" />
+    <joint name="${arm_prefix}suction_gripper_attaching_point_joint" type="fixed">
         <parent link="${arm_prefix}flange_rotated_link"/>
-        <child link="${arm_prefix}suction_gripper_mount_frame"/>
-        <origin xyz="0.065141 0.0 -0.03299" rpy="0 ${pi/2 + pi/3} 0"/>
+        <child link="${arm_prefix}suction_gripper_attaching_point"/>
+        <origin xyz="0.052123 0.0 -0.037123" rpy="0 ${pi/2 + pi/4} 0"/>
     </joint>
     <!-- add suction gripper  -->
@@ -135,5 +139,5 @@
     </link>
     <joint name="${arm_prefix}suction_gripper_joint" type="fixed">
-        <parent link="${arm_prefix}suction_gripper_mount_frame"/>
+        <parent link="${arm_prefix}suction_gripper_attaching_point"/>
         <child link="${arm_prefix}suction_gripper"/>
         <origin xyz="0.0 0.0 -0.0065" rpy="0 0 0"/>
@@ -142,5 +146,5 @@
     <link name="${arm_prefix}suction_tcp" />
     <joint name="${arm_prefix}suction_tcp_joint" type="fixed">
-        <parent link="${arm_prefix}suction_gripper"/>
+        <parent link="${arm_prefix}suction_gripper_attaching_point"/>
         <child link="${arm_prefix}suction_tcp"/>
         <origin xyz="0 0 ${0.144 + thickness_of_the_suction_cup}" rpy="0 0 0"/>
@@ -174,5 +178,5 @@
     <xacro:property name="rail_length" value="2.0"/>
     <xacro:property name="rail_width" value="0.8"/>
-    <xacro:property name="rail_height" value="0.8"/>
+    <xacro:property name="rail_height" value="0.745"/>
     <link name="rail_link">
         <visual>
@@ -198,5 +202,5 @@
         <parent link="world"/>
         <child link="rail_link"/>
-        <origin xyz="${rail_width/2 + 0.1} ${0/2} ${-rail_height/2 - 0.1}" rpy="0 0 ${pi/2}"/>
+        <origin xyz="${rail_width/2 + 0.1} ${0/2} ${-cobot_station_height+rail_height/2}" rpy="0 0 ${pi/2}"/>
     </joint>
 </robot>

Commit message: correct the robot pose in world

File: src/wrs_cell_description/urdf/wrs_env_V2.urdf.xacro (robot description, xacro)
@@ -29,5 +29,5 @@
         visual_parameters_file="$(find ur_description)/config/ur5e/visual_parameters.yaml"
         initial_positions="${initial_positions}">
-        <origin xyz="${-0.27/2} ${-0.27/2} 0.015" rpy="0 0 ${pi}"/>
+        <origin xyz="${-0.27/2} -.012 0.015" rpy="0 0 ${pi}"/>
     </xacro:ur_robot>
     <!-- World link -->

Commit message: change the color of 3d printed parts to dark gray

File: src/wrs_cell_description/urdf/wrs_env_V2.urdf.xacro (robot description, xacro)
@@ -68,4 +68,7 @@
           <mesh filename="package://robot_description/meshes/gripper_adapter.stl" scale="0.001 0.001 0.001"/>
         </geometry>
+        <material name="dark_grey">
+          <color rgba="0.3 0.3 0.3 1.0"/>
+        </material>
       </visual>
       <collision>
@@ -125,4 +128,7 @@
                 <mesh filename="package://robot_description/meshes/suction_gripper/visual/suction_gripper.stl" />
             </geometry>
+            <material name="dark_grey">
+            <color rgba="0.3 0.3 0.3 1.0"/>
+            </material>
         </visual>
         <collision>

Commit message: add new suction cup holder + suction cups meshes

File: src/wrs_cell_description/urdf/wrs_env_V2.urdf.xacro (robot description, xacro)
@@ -126,5 +126,6 @@
         <visual>
             <geometry>
-                <mesh filename="package://robot_description/meshes/suction_gripper/visual/suction_gripper.stl" />
+                <!-- <mesh filename="package://robot_description/meshes/suction_gripper/visual/SuctionCupHolder.stl" scale="0.001 0.001 0.001" /> -->
+                <mesh filename="package://robot_description/meshes/suction_gripper/visual/SuctionCupHolder.dae" />
             </geometry>
             <material name="dark_grey">
@@ -134,5 +135,5 @@
         <collision>
             <geometry>
-                <mesh filename="package://robot_description/meshes/suction_gripper/collision/suction_gripper.stl" />
+                <mesh filename="package://robot_description/meshes/suction_gripper/collision/SuctionCupHolder.stl"/>
             </geometry>
         </collision>
@@ -147,5 +148,5 @@
         <parent link="${arm_prefix}suction_gripper_attaching_point"/>
         <child link="${arm_prefix}suction_gripper"/>
-        <origin xyz="0.0 0.0 -0.0065" rpy="0 0 0"/>
+        <origin xyz="0.0 0.0 0.0" rpy="0 0 ${pi/2}"/>
     </joint>
     <!-- Suction Cup Tool Center Point (TCP) - Frame between suction cup -->

Commit message: add visual mesh for robotiq coupler

File: src/wrs_cell_description/urdf/wrs_env_V2.urdf.xacro (robot description, xacro)
@@ -91,4 +91,16 @@
     <!-- ======================================== Robotiq gripper ======================================== -->
     <link name="${arm_prefix}robotiq_attaching_point" />
+    <link name="${arm_prefix}robotiq_coupler_link" >
+        <visual>
+            <geometry>
+                <mesh filename="package://robot_description/meshes/RobotiqCoupler.dae" />
+            </geometry>
+        </visual>
+    </link>
+    <joint name="${arm_prefix}robotiq_coupler_joint" type="fixed">
+        <parent link="${arm_prefix}robotiq_attaching_point"/>
+        <child link="${arm_prefix}robotiq_coupler_link"/>
+        <origin xyz="0 0 0" rpy="0 ${pi/2} 0"/>
+    </joint>
     <!-- gripper tcp offset - from base of the robotiq to tip of the fingers in closed position -->
     <!-- reference: https://assets.robotiq.com/website-assets/support_documents/document/online/2F-85_2F-140_TM_InstructionManual_HTML5_20190503.zip/2F-85_2F-140_TM_InstructionManual_HTML5/Content/6.%20Specifications.htm -->

Commit message: corrected the ur5_suction_tcp offset

File: src/wrs_cell_description/urdf/wrs_env_V2.urdf.xacro (robot description, xacro)
@@ -7,5 +7,5 @@
     <xacro:arg name="robot_ip" default="192.168.1.102"/>
     <!-- suction gripper properties -->
-    <xacro:property name="thickness_of_the_suction_cup" value="0.030" /> <!-- 30mm -->
+    <xacro:property name="thickness_of_the_suction_cup" value="0.016" /> <!-- 16mm -->
     <!-- Include official UR5e description from ur_description package -->
     <xacro:include filename="$(find ur_description)/urdf/ur_macro.xacro"/>
@@ -167,5 +167,5 @@
         <parent link="${arm_prefix}suction_gripper_attaching_point"/>
         <child link="${arm_prefix}suction_tcp"/>
-        <origin xyz="0 0 ${0.144 + thickness_of_the_suction_cup}" rpy="0 0 0"/>
+        <origin xyz="0 0 ${0.084 + thickness_of_the_suction_cup}" rpy="0 0 0"/>
     </joint>
     <!-- add camera pillar -->

Commit message: corrected the suction cup thicknesses

File: src/wrs_cell_description/urdf/wrs_env_V2.urdf.xacro (robot description, xacro)
@@ -7,5 +7,5 @@
     <xacro:arg name="robot_ip" default="192.168.1.102"/>
     <!-- suction gripper properties -->
-    <xacro:property name="thickness_of_the_suction_cup" value="0.016" /> <!-- 16mm -->
+    <xacro:property name="thickness_of_the_suction_cup" value="0.035" /> <!-- 35mm -->
     <!-- Include official UR5e description from ur_description package -->
     <xacro:include filename="$(find ur_description)/urdf/ur_macro.xacro"/>
