Commit message: - Resolved unrealistic inertia of robtiq gripper parts

File: src/robot_description/urdf/robotiq/robotiq_85_gripper.urdf.xacro (robot description, xacro)
@@ -55,7 +55,7 @@
         <mass value="0.018491" />
         <origin xyz="0.0 0.0 0.0" />
-        <inertia ixx = "0.000009" ixy = "-0.000001" ixz = "0.000000"
-             iyx = "-0.000001" iyy = "0.000001" iyz = "0.000000"
-             izx = "0.000000" izy = "0.000000" izz = "0.000010" />
+        <inertia ixx = "0.000009" ixy = "0.0" ixz = "0.0"
+             iyx = "0.0" iyy = "0.000007" iyz = "0.0"
+             izx = "0.0" izy = "0.0" izz = "0.000010" />
       </inertial>
     </link>
@@ -74,7 +74,7 @@
         <mass value="0.018491" />
         <origin xyz="0.0 0.0 0.0" />
-        <inertia ixx = "0.000009" ixy = "-0.000001" ixz = "0.000000"
-             iyx = "-0.000001" iyy = "0.000001" iyz = "0.000000"
-             izx = "0.000000" izy = "0.000000" izz = "0.000010" />
+        <inertia ixx = "0.000009" ixy = "0.0" ixz = "0.0"
+             iyx = "0.0" iyy = "0.000007" iyz = "0.0"
+             izx = "0.0" izy = "0.0" izz = "0.000010" />
       </inertial>
     </link>
