Commit message: fix moveit

File: src/wrs_env_v2_moveit_config/config/wrs_cell_v2.ros2_control.xacro (robot description, xacro)
@@ -8,4 +8,11 @@
                 <plugin>mock_components/GenericSystem</plugin>
             </hardware>
+            <joint name="ur5_robotiq_85_left_knuckle_joint">
+                <command_interface name="position"/>
+                <state_interface name="position">
+                  <param name="initial_value">${initial_positions['ur5_robotiq_85_left_knuckle_joint']}</param>
+                </state_interface>
+                <state_interface name="velocity"/>
+            </joint>
             <joint name="ur5_shoulder_pan_joint">
                 <command_interface name="position"/>
@@ -50,11 +57,4 @@
                 <state_interface name="velocity"/>
             </joint>
-            <joint name="ur5_robotiq_85_left_knuckle_joint">
-                <command_interface name="position"/>
-                <state_interface name="position">
-                  <param name="initial_value">${initial_positions['ur5_robotiq_85_left_knuckle_joint']}</param>
-                </state_interface>
-                <state_interface name="velocity"/>
-            </joint>
         </ros2_control>
     </xacro:macro>
